File: untitled.kicad_sch (KiCad schematic)
At the start: 12 parts, among them J5 Screw_Terminal_01x02, U3 LM2596S-ADJ, U4 TPS54560BDDA

Commit message: Autosave
Connections:
- net at R9.1: now also U4.2 (VIN)
Other:
- moved on the sheet: R9
Changed lines of the file:
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@@
+	(wire
+		(pts
+			(xy 69.85 38.1) (xy 80.01 38.1)
+		)
+		(stroke
+			(width 0)
+			(type default)
+		)
+	)
 	(wire
 		(pts
@@
 	(symbol
 		(lib_id "Device:R")
-		(at 44.45 41.91 0)
+		(at 69.85 41.91 0)
 		(unit 1)
 		(body_style 1)
@@
 		(fields_autoplaced yes)
 		(property "Reference" "R9"
-			(at 46.99 40.6399 0)
+			(at 72.39 40.6399 0)
 			(show_name no)
 			(do_not_autoplace no)
@@
 		)
 		(property "Value" "1k"
-			(at 46.99 43.1799 0)
+			(at 72.39 43.1799 0)
 			(show_name no)
 			(do_not_autoplace no)
@@
 		)
 		(property "Footprint" ""
-			(at 42.672 41.91 90)
+			(at 68.072 41.91 90)
 			(hide yes)
 			(show_name no)
@@
 		)
 		(property "Datasheet" ""
-			(at 44.45 41.91 0)
+			(at 69.85 41.91 0)
 			(hide yes)
 			(show_name no)
@@
 		)
 		(property "Description" "Resistor"
-			(at 44.45 41.91 0)
-			(hide yes)
-			(show_name no)
+			(at 69.85 41.91 0)
+			(hide yes)
+			(show_name no)

Commit message: Autosave
Connections:
- net at R9.2: now also U4.3 (EN)
Changed lines of the file:
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@@
+	(wire
+		(pts
+			(xy 73.66 45.72) (xy 73.66 43.18)
+		)
+		(stroke
+			(width 0)
+			(type default)
+		)
+	)
 	(wire
 		(pts
@@
 	(wire
 		(pts
+			(xy 73.66 43.18) (xy 80.01 43.18)
+		)
+		(stroke
+			(width 0)
+			(type default)
+		)
+	)
+	(wire
+		(pts
 			(xy 231.14 27.94) (xy 231.14 25.4)
 		)
@@
 		)
 		(stroke
+			(width 0)
+			(type default)
+		)
+	)
+	(wire
+		(pts
+			(xy 69.85 45.72) (xy 73.66 45.72)
+		)
+		(stroke

Commit message: Autosave
Parts:
- R9: value 1k -> 442k
Changed lines of the file:
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@@
 			)
 		)
-		(property "Value" "1k"
+		(property "Value" "442k"
 			(at 72.39 43.1799 0)
 			(show_name no)

Commit message: Autosave
Parts:
- added R11: 442k, symbol Device:R
Changed lines of the file:
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@@
 		(in_pos_files yes)
 		(dnp no)
-		(fields_autoplaced yes)
 		(property "Reference" "R9"
 			(at 72.39 40.6399 0)
@@
 		)
 		(property "Value" "442k"
-			(at 72.39 43.1799 0)
+			(at 64.008 41.148 0)
 			(show_name no)
 			(do_not_autoplace no)
@@
 					(unit 1)
 				)
+			)
+		)
+	)
+	(symbol
+		(lib_id "Device:R")
+		(at 69.85 52.07 0)
+		(unit 1)
+		(body_style 1)
+		(exclude_from_sim no)
+		(in_bom yes)
+		(on_board yes)
+		(in_pos_files yes)
+		(dnp no)
+		(property "Reference" "R11"
+			(at 72.39 50.7999 0)
+			(show_name no)
+			(do_not_autoplace no)
+			(effects
+				(font
+					(size 1.27 1.27)
+				)
+				(justify left)
+			)
+		)
+		(property "Value" "442k"
+			(at 64.008 51.308 0)
+			(show_name no)
+			(do_not_autoplace no)
+			(effects
+				(font
+					(size 1.27 1.27)
+				)
+				(justify left)
+			)
+		)
+		(property "Footprint" ""
+			(at 68.072 52.07 90)
+			(hide yes)
+			(show_name no)
+			(do_not_autoplace no)
+			(effects
+				(font
+					(size 1.27 1.27)
+				)
+			)
+		)
+		(property "Datasheet" ""
+			(at 69.85 52.07 0)
+			(hide yes)
+			(show_name no)
+			(do_not_autoplace no)
+			(effects
+				(font
+					(size 1.27 1.27)
+				)
+			)
+		)
+		(property "Description" "Resistor"
+			(at 69.85 52.07 0)
+			(hide yes)
+			(show_name no)
+			(do_not_autoplace no)
+			(effects
+				(font
+					(size 1.27 1.27)
+				)
+			)
+		)
+		(pin "1"
+		)
+		(pin "2"
+		)
+		(instances
+			(project "flight controller"
+				(path "/d0cd3d3b-d42f-4a0d-9317-17db4a7f672b/01eadb20-ad5a-457b-b9aa-f1bf9fe7a694"
+					(reference "R11")
+					(unit 1)
+				)

Commit message: Autosave
Parts:
- added R12: 442k, symbol Device:R
Connections:
- net at R9.2, U4.3 (EN): now also R11.1
Other:
- moved on the sheet: R11
Changed lines of the file:
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@@
+	)
+	(junction
+		(at 69.85 45.72)
+		(diameter 0)
+		(color 0 0 0 0)
 	)
 	(junction
@@
 	)
 	(symbol
+		(lib_id "Device:R")
+		(at 78.74 53.34 0)
+		(unit 1)
+		(body_style 1)
+		(exclude_from_sim no)
+		(in_bom yes)
+		(on_board yes)
+		(in_pos_files yes)
+		(dnp no)
+		(property "Reference" "R12"
+			(at 81.28 52.0699 0)
+			(show_name no)
+			(do_not_autoplace no)
+			(effects
+				(font
+					(size 1.27 1.27)
+				)
+				(justify left)
+			)
+		)
+		(property "Value" "442k"
+			(at 72.898 52.578 0)
+			(show_name no)
+			(do_not_autoplace no)
+			(effects
+				(font
+					(size 1.27 1.27)
+				)
+				(justify left)
+			)
+		)
+		(property "Footprint" ""
+			(at 76.962 53.34 90)
+			(hide yes)
+			(show_name no)
+			(do_not_autoplace no)
+			(effects
+				(font
+					(size 1.27 1.27)
+				)
+			)
+		)
+		(property "Datasheet" ""
+			(at 78.74 53.34 0)
+			(hide yes)
+			(show_name no)
+			(do_not_autoplace no)
+			(effects
+				(font
+					(size 1.27 1.27)
+				)
+			)
+		)
+		(property "Description" "Resistor"
+			(at 78.74 53.34 0)
+			(hide yes)
+			(show_name no)
+			(do_not_autoplace no)
+			(effects
+				(font
+					(size 1.27 1.27)
+				)
+			)
+		)
+		(pin "1"
+		)
+		(pin "2"
+		)
+		(instances
+			(project "flight controller"
+				(path "/d0cd3d3b-d42f-4a0d-9317-17db4a7f672b/01eadb20-ad5a-457b-b9aa-f1bf9fe7a694"
+					(reference "R12")
+					(unit 1)
+				)
+			)
+		)
+	)
+	(symbol
 		(lib_id "Diode:SS34")
 		(at 90.17 92.71 0)
@@
 	(symbol
 		(lib_id "Device:R")
-		(at 69.85 52.07 0)
+		(at 69.85 49.53 0)
 		(unit 1)
 		(body_style 1)
@@
 		(dnp no)
 		(property "Reference" "R11"
-			(at 72.39 50.7999 0)
+			(at 72.39 48.2599 0)
 			(show_name no)
 			(do_not_autoplace no)
@@
 		)
 		(property "Value" "442k"
-			(at 64.008 51.308 0)
+			(at 64.008 48.768 0)
 			(show_name no)
 			(do_not_autoplace no)
@@
 		)
 		(property "Footprint" ""
-			(at 68.072 52.07 90)
+			(at 68.072 49.53 90)
 			(hide yes)
 			(show_name no)
@@
 		)
 		(property "Datasheet" ""
-			(at 69.85 52.07 0)
+			(at 69.85 49.53 0)
 			(hide yes)
 			(show_name no)
@@
 		)
 		(property "Description" "Resistor"
-			(at 69.85 52.07 0)
-			(hide yes)
-			(show_name no)
+			(at 69.85 49.53 0)
+			(hide yes)
+			(show_name no)

Commit message: Autosave
Connections:
- net at R12.1: now also U4.4 (RT/CLK)
Other:
- moved on the sheet: R12
Changed lines of the file:
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@@
 	(symbol
 		(lib_id "Device:R")
-		(at 78.74 53.34 0)
+		(at 80.01 52.07 0)
 		(unit 1)
 		(body_style 1)
@@
 		(dnp no)
 		(property "Reference" "R12"
-			(at 81.28 52.0699 0)
+			(at 81.534 52.578 0)
 			(show_name no)
 			(do_not_autoplace no)
@@
 		)
 		(property "Value" "442k"
-			(at 72.898 52.578 0)
+			(at 74.168 51.308 0)
 			(show_name no)
 			(do_not_autoplace no)
@@
 		)
 		(property "Footprint" ""
-			(at 76.962 53.34 90)
+			(at 78.232 52.07 90)
 			(hide yes)
 			(show_name no)
@@
 		)
 		(property "Datasheet" ""
-			(at 78.74 53.34 0)
+			(at 80.01 52.07 0)
 			(hide yes)
 			(show_name no)
@@
 		)
 		(property "Description" "Resistor"
-			(at 78.74 53.34 0)
+			(at 80.01 52.07 0)
 			(hide yes)
 			(show_name no)

Commit message: Autosave
Parts:
- R12: value 442k -> 243k
Changed lines of the file:
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@@
 			)
 		)
-		(property "Value" "442k"
+		(property "Value" "243k"
 			(at 74.168 51.308 0)
 			(show_name no)

Commit message: Autosave
Parts:
- R11: value 442k -> 90.9k
Other:
- moved on the sheet: R11
Changed lines of the file:
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@@
-	)
-	(junction
-		(at 69.85 45.72)
-		(diameter 0)
-		(color 0 0 0 0)
 	)
 	(junction
@@
 		(pts
 			(xy 274.32 25.4) (xy 274.32 30.48)
+		)
+		(stroke
+			(width 0)
+			(type default)
+		)
+	)
+	(wire
+		(pts
+			(xy 69.85 46.99) (xy 69.85 45.72)
 		)
 		(stroke
@@
 	(symbol
 		(lib_id "Device:R")
-		(at 69.85 49.53 0)
+		(at 69.85 50.8 0)
 		(unit 1)
 		(body_style 1)
@@
 		(dnp no)
 		(property "Reference" "R11"
-			(at 72.39 48.2599 0)
-			(show_name no)
-			(do_not_autoplace no)
-			(effects
-				(font
-					(size 1.27 1.27)
-				)
-				(justify left)
-			)
-		)
-		(property "Value" "442k"
-			(at 64.008 48.768 0)
+			(at 72.39 49.5299 0)
+			(show_name no)
+			(do_not_autoplace no)
+			(effects
+				(font
+					(size 1.27 1.27)
+				)
+				(justify left)
+			)
+		)
+		(property "Value" "90.9k"
+			(at 64.008 50.038 0)
 			(show_name no)
 			(do_not_autoplace no)
@@
 		)
 		(property "Footprint" ""
-			(at 68.072 49.53 90)
+			(at 68.072 50.8 90)
 			(hide yes)
 			(show_name no)
@@
 		)
 		(property "Datasheet" ""
-			(at 69.85 49.53 0)
+			(at 69.85 50.8 0)
 			(hide yes)
 			(show_name no)
@@
 		)
 		(property "Description" "Resistor"
-			(at 69.85 49.53 0)
-			(hide yes)
-			(show_name no)
+			(at 69.85 50.8 0)
+			(hide yes)
+			(show_name no)
