File: untitled.kicad_sch (KiCad schematic)
At the start: 24 parts, among them J5 Screw_Terminal_01x02, U3 LM2596S-ADJ, U4 TPS54560BDDA

Commit message: Autosave
Parts:
- C24: value 2.2uf -> 47uf
Changed lines of the file:
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@@
 			)
 		)
-		(property "Value" "2.2uf"
+		(property "Value" "47uf"
 			(at 133.096 33.02 0)
 			(show_name no)

Commit message: Autosave
Parts:
- C25: value 2.2uf -> 47uf
Changed lines of the file:
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@@
 			)
 		)
-		(property "Value" "2.2uf"
+		(property "Value" "47uf"
 			(at 144.526 33.02 0)
 			(show_name no)

Commit message: Autosave
Parts:
- C26: value 2.2uf -> 47uf
Changed lines of the file:
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@@
 			)
 		)
-		(property "Value" "2.2uf"
+		(property "Value" "47uf"
 			(at 156.972 33.02 0)
 			(show_name no)

Commit message: Autosave
Parts:
- added L2: 33uh, symbol Device:L
Changed lines of the file:
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@@
+		)
+	)
+	(symbol
+		(lib_id "Device:L")
+		(at 125.73 26.67 90)
+		(unit 1)
+		(body_style 1)
+		(exclude_from_sim no)
+		(in_bom yes)
+		(on_board yes)
+		(in_pos_files yes)
+		(dnp no)
+		(property "Reference" "L2"
+			(at 122.428 24.638 90)
+			(show_name no)
+			(do_not_autoplace no)
+			(effects
+				(font
+					(size 1.27 1.27)
+				)
+			)
+		)
+		(property "Value" "33uh"
+			(at 126.238 24.384 90)
+			(show_name no)
+			(do_not_autoplace no)
+			(effects
+				(font
+					(size 1.27 1.27)
+				)
+			)
+		)
+		(property "Footprint" ""
+			(at 125.73 26.67 0)
+			(hide yes)
+			(show_name no)
+			(do_not_autoplace no)
+			(effects
+				(font
+					(size 1.27 1.27)
+				)
+			)
+		)
+		(property "Datasheet" ""
+			(at 125.73 26.67 0)
+			(hide yes)
+			(show_name no)
+			(do_not_autoplace no)
+			(effects
+				(font
+					(size 1.27 1.27)
+				)
+			)
+		)
+		(property "Description" "Inductor"
+			(at 125.73 26.67 0)
+			(hide yes)
+			(show_name no)
+			(do_not_autoplace no)
+			(effects
+				(font
+					(size 1.27 1.27)
+				)
+			)
+		)
+		(pin "2"
+		)
+		(pin "1"
+		)
+		(instances
+			(project "flight controller"
+				(path "/d0cd3d3b-d42f-4a0d-9317-17db4a7f672b/01eadb20-ad5a-457b-b9aa-f1bf9fe7a694"
+					(reference "L2")
+					(unit 1)
+				)
+			)
 		)
 	)

Commit message: Autosave
Parts:
- L2: value 33uh -> 7.2uh
Changed lines of the file:
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@@
 			)
 		)
-		(property "Value" "33uh"
+		(property "Value" "7.2uh"
 			(at 126.238 24.384 90)
 			(show_name no)

Commit message: Autosave
Parts:
- added R14, R15: 90.9k, symbol Device:R
Changed lines of the file:
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@@
+	)
+	(symbol
+		(lib_id "Device:R")
+		(at 168.91 38.1 0)
+		(unit 1)
+		(body_style 1)
+		(exclude_from_sim no)
+		(in_bom yes)
+		(on_board yes)
+		(in_pos_files yes)
+		(dnp no)
+		(property "Reference" "R14"
+			(at 170.434 35.56 0)
+			(show_name no)
+			(do_not_autoplace no)
+			(effects
+				(font
+					(size 1.27 1.27)
+				)
+				(justify left)
+			)
+		)
+		(property "Value" "90.9k"
+			(at 162.306 38.608 0)
+			(show_name no)
+			(do_not_autoplace no)
+			(effects
+				(font
+					(size 1.27 1.27)
+				)
+				(justify left)
+			)
+		)
+		(property "Footprint" ""
+			(at 167.132 38.1 90)
+			(hide yes)
+			(show_name no)
+			(do_not_autoplace no)
+			(effects
+				(font
+					(size 1.27 1.27)
+				)
+			)
+		)
+		(property "Datasheet" ""
+			(at 168.91 38.1 0)
+			(hide yes)
+			(show_name no)
+			(do_not_autoplace no)
+			(effects
+				(font
+					(size 1.27 1.27)
+				)
+			)
+		)
+		(property "Description" "Resistor"
+			(at 168.91 38.1 0)
+			(hide yes)
+			(show_name no)
+			(do_not_autoplace no)
+			(effects
+				(font
+					(size 1.27 1.27)
+				)
+			)
+		)
+		(pin "1"
+		)
+		(pin "2"
+		)
+		(instances
+			(project "flight controller"
+				(path "/d0cd3d3b-d42f-4a0d-9317-17db4a7f672b/01eadb20-ad5a-457b-b9aa-f1bf9fe7a694"
+					(reference "R14")
+					(unit 1)
+				)
+			)
+		)
 	)
 	(symbol
@@
 					(unit 1)
 				)
+			)
+		)
+	)
+	(symbol
+		(lib_id "Device:R")
+		(at 168.91 54.61 0)
+		(unit 1)
+		(body_style 1)
+		(exclude_from_sim no)
+		(in_bom yes)
+		(on_board yes)
+		(in_pos_files yes)
+		(dnp no)
+		(property "Reference" "R15"
+			(at 170.434 52.07 0)
+			(show_name no)
+			(do_not_autoplace no)
+			(effects
+				(font
+					(size 1.27 1.27)
+				)
+				(justify left)
+			)
+		)
+		(property "Value" "90.9k"
+			(at 162.306 55.118 0)
+			(show_name no)
+			(do_not_autoplace no)
+			(effects
+				(font
+					(size 1.27 1.27)
+				)
+				(justify left)
+			)
+		)
+		(property "Footprint" ""
+			(at 167.132 54.61 90)
+			(hide yes)
+			(show_name no)
+			(do_not_autoplace no)
+			(effects
+				(font
+					(size 1.27 1.27)
+				)
+			)
+		)
+		(property "Datasheet" ""
+			(at 168.91 54.61 0)
+			(hide yes)
+			(show_name no)
+			(do_not_autoplace no)
+			(effects
+				(font
+					(size 1.27 1.27)
+				)
+			)
+		)
+		(property "Description" "Resistor"
+			(at 168.91 54.61 0)
+			(hide yes)
+			(show_name no)
+			(do_not_autoplace no)
+			(effects
+				(font
+					(size 1.27 1.27)
+				)
+			)
+		)
+		(pin "1"
+		)
+		(pin "2"
+		)
+		(instances
+			(project "flight controller"
+				(path "/d0cd3d3b-d42f-4a0d-9317-17db4a7f672b/01eadb20-ad5a-457b-b9aa-f1bf9fe7a694"
+					(reference "R15")
+					(unit 1)
+				)

Commit message: Autosave
Parts:
- R15: value 90.9k -> 10.2k
Changed lines of the file:
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@@
 			)
 		)
-		(property "Value" "90.9k"
+		(property "Value" "10.2k"
 			(at 162.306 55.118 0)
 			(show_name no)

Commit message: Autosave
Parts:
- R14: value 90.9k -> 53.6k
Other:
- moved on the sheet: R14
Changed lines of the file:
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@@
 	(symbol
 		(lib_id "Device:R")
-		(at 168.91 38.1 0)
+		(at 168.91 40.64 0)
 		(unit 1)
 		(body_style 1)
@@
 		(dnp no)
 		(property "Reference" "R14"
-			(at 170.434 35.56 0)
+			(at 170.434 38.1 0)
 			(show_name no)
 			(do_not_autoplace no)
@@
 			)
 		)
-		(property "Value" "90.9k"
-			(at 162.306 38.608 0)
+		(property "Value" "53.6k"
+			(at 162.306 41.148 0)
 			(show_name no)
 			(do_not_autoplace no)
@@
 		)
 		(property "Footprint" ""
-			(at 167.132 38.1 90)
+			(at 167.132 40.64 90)
 			(hide yes)
 			(show_name no)
@@
 		)
 		(property "Datasheet" ""
-			(at 168.91 38.1 0)
+			(at 168.91 40.64 0)
 			(hide yes)
 			(show_name no)
@@
 		)
 		(property "Description" "Resistor"
-			(at 168.91 38.1 0)
+			(at 168.91 40.64 0)
 			(hide yes)
 			(show_name no)
