File: flight controller.kicad_sch (KiCad schematic)
At the start: 38 parts, among them J1 USB_C_Receptacle_USB2.0_16P, J2 Conn_01x04_Pin, J3 Conn_01x04_Pin, J4 Conn_01x04_Pin, J6 Conn_01x06_Pin, SW1 SW_Push, SW2 SW_SPDT, U1 STM32H743VITx, U2 USBLC6-2SC6, Y1 16MHz

Commit message: Autosave
Other:
- note added: "GPS"
Changed lines of the file:
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@@
+		)
+	)
+	(text "GPS"
+		(exclude_from_sim no)
+		(at 36.068 91.44 0)
+		(effects
+			(font
+				(size 2.54 2.54)
+				(thickness 0.508)
+				(bold yes)
+			)
 		)
 	)

Commit message: Autosave
Connections:
- net pd6: now also U1.87 (PD6)
Changed lines of the file:
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@@
+		)
+	)
+	(label "pd6"
+		(at 120.65 127 180)
+		(effects
+			(font
+				(size 1.27 1.27)
+			)
+			(justify right bottom)
 		)
 	)

Commit message: Autosave
Connections:
- net pd6: no longer names the net of J6.2 (Pin_2)
- net pd6: no longer U1.87 (PD6)
- new net pd6(TX): U1.87 (PD6)
Changed lines of the file:
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@@
 		)
 	)
-	(label "pd6"
-		(at 27.94 104.14 0)
-		(effects
-			(font
-				(size 1.27 1.27)
-			)
-			(justify left bottom)
-		)
-	)
-	(label "pd6"
+	(label "pd6(TX)"
 		(at 120.65 127 180)
 		(effects

Commit message: Autosave
Connections:
- net pd6(TX): now also J6.2 (Pin_2)
Changed lines of the file:
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@@
+		)
+	)
+	(label "pd6(TX)"
+		(at 27.94 104.14 0)
+		(effects
+			(font
+				(size 1.27 1.27)
+			)
+			(justify left bottom)
 		)
 	)

Commit message: Autosave
Connections:
- net pd5 renamed pd5(RX)
Changed lines of the file:
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@@
 		)
 	)
-	(label "pd5"
+	(label "pd5(RX)"
 		(at 27.94 106.68 0)
 		(effects

Commit message: Autosave
Connections:
- net pb10 renamed pb10(SCL)
Changed lines of the file:
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@@
 		)
 	)
-	(label "pb10"
+	(label "pb10(SCL)"
 		(at 27.94 109.22 0)
 		(effects

Commit message: Autosave
Connections:
- net pd5(RX): now also U1.86 (PD5)
- net pb11 renamed pb11(SDA)
Changed lines of the file:
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@@
 		)
 	)
-	(label "pb11"
+	(label "pb11(SDA)"
 		(at 27.94 111.76 0)
 		(effects
@@
 		)
 	)
+	(label "pd5(RX)"
+		(at 120.65 124.46 180)
+		(effects
+			(font
+				(size 1.27 1.27)
+			)
+			(justify right bottom)
+		)
+	)

Commit message: Autosave
Parts:
- removed J3: Conn_01x04_Pin, symbol Connector:Conn_01x04_Pin
