File: flight controller.kicad_sch (KiCad schematic)
At the start: 37 parts, among them J1 USB_C_Receptacle_USB2.0_16P, J2 Conn_01x04_Pin, J4 Conn_01x04_Pin, J6 Conn_01x06_Pin, SW1 SW_Push, SW2 SW_SPDT, U1 STM32H743VITx, U2 USBLC6-2SC6, Y1 16MHz

Commit message: Autosave
Parts:
- R7, R8: value 4.7k -> 2.2K
Changed lines of the file:
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@@
 			)
 		)
-		(property "Value" "4.7k"
+		(property "Value" "2.2K"
 			(at 180.34 121.9199 0)
 			(show_name no)
@@
 			)
 		)
-		(property "Value" "4.7k"
+		(property "Value" "2.2K"
 			(at 172.212 121.666 0)
 			(show_name no)

Commit message: Autosave
Connections:
- net pb10(SCL) is gone; now on net i2c2 scl: J6.4 (Pin_4)
- net pb11(SDA) is gone; now on net i2c2 sda: J6.5 (Pin_5)
Changed lines of the file:
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@@
+		)
+	)
+	(label "pb10(SCL)"
+		(at 187.96 125.73 0)
+		(effects
+			(font
+				(size 1.27 1.27)
+			)
+			(justify left bottom)
 		)
 	)
@@
 		(effects
 			(font
+				(size 1.27 1.27)
+			)
+			(justify left bottom)
+		)
+	)
+	(label "pb11(SDA)"
+		(at 185.42 128.27 0)
+		(effects
+			(font

Commit message: Autosave
Connections:
- net +3.3V: no longer J4.4 (Pin_4)
- new net 3.3V: J4.4 (Pin_4)
Changed lines of the file:
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@@
 			)
 		)
-		(property "Value" "+3.3V"
+		(property "Value" "3.3V"
 			(at 208.28 99.314 0)
 			(show_name no)

Commit message: Autosave
Connections:
- net +3.3V: no longer R5.1, R6.1
- net 3.3V: now also R5.1, R6.1
Changed lines of the file:
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@@
 			)
 		)
-		(property "Value" "+3.3V"
+		(property "Value" "3.3V"
 			(at 176.276 97.79 0)
 			(show_name no)

Commit message: Autosave
Connections:
- net 3.3V: no longer R5.1, R6.1
- new net 3.3v: R5.1, R6.1
Changed lines of the file:
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@@
 			)
 		)
-		(property "Value" "3.3V"
+		(property "Value" "3.3v"
 			(at 176.276 97.79 0)
 			(show_name no)

Commit message: Autosave
Connections:
- net 3.3V is gone; now on net 3.3v: J4.4 (Pin_4)
Changed lines of the file:
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@@
 			)
 		)
-		(property "Value" "3.3V"
+		(property "Value" "3.3v"
 			(at 208.28 99.314 0)
 			(show_name no)

Commit message: Autosave
Parts:
- removed J1: USB_C_Receptacle_USB2.0_16P, Connector_USB:USB_C_Receptacle_Amphenol_12401548E4-2A, symbol Connector:USB_C_Receptacle_USB2.0_16P
Connections:
- net +3.3V: no longer R4.2
- no-connect marks 2 -> 0
Changed lines of the file:
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@@
 	)
 	(junction
-		(at 236.22 45.72)
-		(diameter 0)
-		(color 0 0 0 0)
-	)
-	(junction
 		(at 138.43 31.75)
 		(diameter 0)
@@
 	)
 	(junction
-		(at 243.84 45.72)
-		(diameter 0)
-		(color 0 0 0 0)
-	)
-	(junction
 		(at 73.66 35.56)
 		(diameter 0)
@@
 		(color 0 0 0 0)
 	)
-	(no_connect
-		(at 220.98 53.34)
-	)
-	(no_connect
-		(at 220.98 55.88)
-	)
 	(wire
 		(pts
@@
 	(wire
 		(pts
-			(xy 204.47 45.72) (xy 236.22 45.72)
-		)
-		(stroke
-			(width 0)
-			(type default)
-		)
-	)
-	(wire
-		(pts
 			(xy 92.71 45.72) (xy 95.25 45.72)
 		)
@@
 	(wire
 		(pts
-			(xy 236.22 45.72) (xy 243.84 45.72)
+			(xy 204.47 45.72) (xy 243.84 45.72)
 		)
 		(stroke
@@
 	(wire
 		(pts
-			(xy 193.04 54.61) (xy 193.04 57.15)
-		)
-		(stroke
-			(width 0)
-			(type default)
-		)
-	)
-	(wire
-		(pts
 			(xy 134.62 26.67) (xy 134.62 27.94)
 		)
@@
 	(symbol
 		(lib_id "power:+3.3V")
-		(at 193.04 54.61 0)
-		(unit 1)
-		(body_style 1)
-		(exclude_from_sim no)
-		(in_bom yes)
-		(on_board yes)
-		(in_pos_files yes)
-		(dnp no)
-		(fields_autoplaced yes)
-		(property "Reference" "#PWR019"
-			(at 193.04 58.42 0)
-			(hide yes)
-			(show_name no)
-			(do_not_autoplace no)
-			(effects
-				(font
-					(size 1.27 1.27)
-				)
-			)
-		)
-		(property "Value" "+3.3V"
-			(at 193.04 49.53 0)
-			(show_name no)
-			(do_not_autoplace no)
-			(effects
-				(font
-					(size 1.27 1.27)
-				)
-			)
-		)
-		(property "Footprint" ""
-			(at 193.04 54.61 0)
-			(hide yes)
-			(show_name no)
-			(do_not_autoplace no)
-			(effects
-				(font
-					(size 1.27 1.27)
-				)
-			)
-		)
-		(property "Datasheet" ""
-			(at 193.04 54.61 0)
-			(hide yes)
-			(show_name no)
-			(do_not_autoplace no)
-			(effects
-				(font
-					(size 1.27 1.27)
-				)
-			)
-		)
-		(property "Description" "Power symbol creates a global label with name \"+3.3V\""
-			(at 193.04 54.61 0)
-			(hide yes)
-			(show_name no)
-			(do_not_autoplace no)
-			(effects
-				(font
-					(size 1.27 1.27)
-				)
-			)
-		)
-		(pin "1"
-		)
-		(instances
-			(project "flight controller"
-				(path "/d0cd3d3b-d42f-4a0d-9317-17db4a7f672b"
-					(reference "#PWR019")
-					(unit 1)
-				)
-			)
-		)
-	)
-	(symbol
-		(lib_id "power:+3.3V")
 		(at 204.47 100.33 0)
 		(unit 1)
@@
 	)
 	(symbol
-		(lib_id "Connector:USB_C_Receptacle_USB2.0_16P")
-		(at 236.22 68.58 180)
-		(unit 1)
-		(body_style 1)
-		(exclude_from_sim no)
-		(in_bom yes)
-		(on_board yes)
-		(in_pos_files yes)
-		(dnp no)
-		(property "Reference" "J1"
-			(at 236.22 91.44 0)
-			(show_name no)
-			(do_not_autoplace no)
-			(effects
-				(font
-					(size 1.27 1.27)
-				)
-			)
-		)
-		(property "Value" "USB_C_Receptacle_USB2.0_16P"
-			(at 236.22 88.9 0)
-			(show_name no)
-			(do_not_autoplace no)
-			(effects
-				(font
-					(size 1.27 1.27)
-				)
-			)
-		)
-		(property "Footprint" "Connector_USB:USB_C_Receptacle_Amphenol_12401548E4-2A"
-			(at 232.41 68.58 0)
-			(hide yes)
-			(show_name no)
-			(do_not_autoplace no)
-			(effects
-				(font
-					(size 1.27 1.27)
-				)
-			)
-		)
-		(property "Datasheet" "https://www.usb.org/sites/default/files/documents/usb_type-c.zip"
-			(at 232.41 68.58 0)
-			(hide yes)
-			(show_name no)
-			(do_not_autoplace no)
-			(effects
-				(font
-					(size 1.27 1.27)
-				)
-			)
-		)
-		(property "Description" "USB 2.0-only 16P Type-C Receptacle connector"
-			(at 236.22 68.58 0)
-			(hide yes)
-			(show_name no)
-			(do_not_autoplace no)
-			(effects
-				(font
-					(size 1.27 1.27)
-				)
-			)
-		)
-		(pin "A9"
-		)
-		(pin "B5"
-		)
-		(pin "A1"
-		)
-		(pin "A4"
-		)
-		(pin "B6"
-		)
-		(pin "B9"
-		)
-		(pin "B8"
-		)
-		(pin "A7"
-		)
-		(pin "A8"
-		)
-		(pin "A12"
-		)
-		(pin "A6"
-		)
-		(pin "B4"
-		)
-		(pin "B7"
-		)
-		(pin "B12"
-		)
-		(pin "SH"
-		)
-		(pin "A5"
-		)
-		(pin "B1"
-		)
-		(instances
-			(project "flight controller"
-				(path "/d0cd3d3b-d42f-4a0d-9317-17db4a7f672b"
-					(reference "J1")
-					(unit 1)
-				)
-			)
-		)
-	)
-	(symbol
 		(lib_id "power:GND")
 		(at 27.94 114.3 90)
@@
 		(property "Reference" "U2"
 			(at 202.8189 57.15 0)
+			(hide yes)
 			(show_name no)
 			(do_not_autoplace no)

Commit message: Autosave
Connections:
- net GND: no longer U2.5 (VBUS)
Changed lines of the file:
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@@
 	(wire
 		(pts
-			(xy 204.47 59.69) (xy 204.47 45.72)
-		)
-		(stroke
-			(width 0)
-			(type default)
-		)
-	)
-	(wire
-		(pts
 			(xy 185.42 91.44) (xy 176.53 91.44)
 		)
@@
 	(wire
 		(pts
-			(xy 204.47 45.72) (xy 243.84 45.72)
-		)
-		(stroke
-			(width 0)
-			(type default)
-		)
-	)
-	(wire
-		(pts
 			(xy 120.65 154.94) (xy 116.84 154.94)
 		)
@@
 	(wire
 		(pts
-			(xy 243.84 40.64) (xy 243.84 45.72)
-		)
-		(stroke
-			(width 0)
-			(type default)
-		)
-	)
-	(wire
-		(pts
 			(xy 220.98 69.85) (xy 220.98 71.12)
 		)
@@
 		(property "Value" "22"
 			(at 195.326 60.706 90)
+			(hide yes)
 			(show_name no)
 			(do_not_autoplace no)
@@
 					(unit 1)
 				)
-			)
-		)
-	)
-	(symbol
-		(lib_id "power:GND")
-		(at 243.84 40.64 180)
-		(unit 1)
-		(body_style 1)
-		(exclude_from_sim no)
-		(in_bom yes)
-		(on_board yes)
-		(in_pos_files yes)
-		(dnp no)
-		(fields_autoplaced yes)
-		(property "Reference" "#PWR018"
-			(at 243.84 34.29 0)
-			(hide yes)
-			(show_name no)
-			(do_not_autoplace no)
-			(effects
-				(font
-					(size 1.27 1.27)
-				)
-			)
-		)
-		(property "Value" "GND"
-			(at 243.84 35.56 0)
-			(show_name no)
-			(do_not_autoplace no)
-			(effects
-				(font
-					(size 1.27 1.27)
-				)
-			)
-		)
-		(property "Footprint" ""
-			(at 243.84 40.64 0)
-			(hide yes)
-			(show_name no)
-			(do_not_autoplace no)
-			(effects
-				(font
-					(size 1.27 1.27)
-				)
-			)
-		)
-		(property "Datasheet" ""
-			(at 243.84 40.64 0)
-			(hide yes)
-			(show_name no)
-			(do_not_autoplace no)
-			(effects
-				(font
-					(size 1.27 1.27)
-				)
-			)
-		)
-		(property "Description" "Power symbol creates a global label with name \"GND\" , ground"
-			(at 243.84 40.64 0)
-			(hide yes)
-			(show_name no)
-			(do_not_autoplace no)
-			(effects
-				(font
-					(size 1.27 1.27)
-				)
-			)
-		)
-		(pin "1"
-		)
-		(instances
-			(project "flight controller"
-				(path "/d0cd3d3b-d42f-4a0d-9317-17db4a7f672b"
-					(reference "#PWR018")
-					(unit 1)
-				)
