File: gps.kicad_sch (KiCad schematic)
At the start: 30 parts, among them J5 Micro_SD_Card_Det_Hirose_DM3AT, U10 TPS54560BDDA, U9 74AHCT125

Commit message: Autosave
Parts:
- added U11: 74AHCT125, symbol symbols:74AHCT125
Connections:
- net 5v: now also U11.14 (VCC)
- net GND: now also U11.1, U11.10, U11.13, U11.4, U11.7 (GND)
- net pa0: now also U11.2
- net pa1: now also U11.5
- net pa2: now also U11.9
- net pa3: now also U11.12
- net s1: now also U11.3
- net s2: now also U11.6
- net s3: now also U11.8
- net s4: now also U11.11

Commit message: Autosave
Connections:
- net s1: no longer U11.3
- net s2: no longer U11.6
- new net s5: U11.3
- new net s6: U11.6
Changed lines of the file:
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@@
 		)
 	)
-	(label "s2"
+	(label "s6"
 		(at 116.84 46.99 0)
 		(effects
@@
 		)
 	)
-	(label "s1"
+	(label "s5"
 		(at 121.92 24.13 0)
 		(effects

Commit message: Autosave
Connections:
- net s3: no longer U11.8
- net s4: no longer U11.11
- new net s7: U11.8
- new net s8: U11.11
Changed lines of the file:
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@@
 		)
 	)
-	(label "s4"
+	(label "s8"
 		(at 123.19 86.36 0)
 		(effects
@@
 		)
 	)
-	(label "s3"
+	(label "s7"
 		(at 125.73 63.5 0)
 		(effects

Commit message: Autosave
Parts:
- added U12: 74AHCT244, symbol 74xx:74AHCT244
Changed lines of the file:
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@@
+		)
+	)
+	(symbol
+		(lib_id "74xx:74AHCT244")
+		(at 77.47 55.88 0)
+		(unit 1)
+		(body_style 1)
+		(exclude_from_sim no)
+		(in_bom yes)
+		(on_board yes)
+		(in_pos_files yes)
+		(dnp no)
+		(fields_autoplaced yes)
+		(property "Reference" "U12"
+			(at 79.6133 35.56 0)
+			(show_name no)
+			(do_not_autoplace no)
+			(effects
+				(font
+					(size 1.27 1.27)
+				)
+				(justify left)
+			)
+		)
+		(property "Value" "74AHCT244"
+			(at 79.6133 38.1 0)
+			(show_name no)
+			(do_not_autoplace no)
+			(effects
+				(font
+					(size 1.27 1.27)
+				)
+				(justify left)
+			)
+		)
+		(property "Footprint" ""
+			(at 77.47 55.88 0)
+			(hide yes)
+			(show_name no)
+			(do_not_autoplace no)
+			(effects
+				(font
+					(size 1.27 1.27)
+				)
+			)
+		)
+		(property "Datasheet" "https://assets.nexperia.com/documents/data-sheet/74AHC_AHCT244.pdf"
+			(at 77.47 55.88 0)
+			(hide yes)
+			(show_name no)
+			(do_not_autoplace no)
+			(effects
+				(font
+					(size 1.27 1.27)
+				)
+			)
+		)
+		(property "Description" "8-bit Buffer/Line Driver 3-state"
+			(at 77.47 55.88 0)
+			(hide yes)
+			(show_name no)
+			(do_not_autoplace no)
+			(effects
+				(font
+					(size 1.27 1.27)
+				)
+			)
+		)
+		(pin "7"
+		)
+		(pin "8"
+		)
+		(pin "6"
+		)
+		(pin "9"
+		)
+		(pin "16"
+		)
+		(pin "15"
+		)
+		(pin "18"
+		)
+		(pin "1"
+		)
+		(pin "5"
+		)
+		(pin "11"
+		)
+		(pin "17"
+		)
+		(pin "19"
+		)
+		(pin "4"
+		)
+		(pin "14"
+		)
+		(pin "20"
+		)
+		(pin "12"
+		)
+		(pin "10"
+		)
+		(pin "3"
+		)
+		(pin "2"
+		)
+		(pin "13"
+		)
+		(instances
+			(project "flight controller"
+				(path "/d0cd3d3b-d42f-4a0d-9317-17db4a7f672b/144e5f7d-352f-43f0-94c0-d8713d07b695"
+					(reference "U12")
+					(unit 1)
+				)
+			)
 		)
 	)

Commit message: Autosave
Connections:
- net pa0: now also U12.2 (1A0)
- net pa1: now also U12.4 (1A1)
Changed lines of the file:
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@@
+	)
+	(label "pa1"
+		(at 64.77 45.72 180)
+		(effects
+			(font
+				(size 1.27 1.27)
+				(thickness 0.254)
+				(bold yes)
+			)
+			(justify right bottom)
+		)
 	)
 	(label "pa1"
@@
 		(effects
 			(font
+				(size 1.27 1.27)
+				(thickness 0.254)
+				(bold yes)
+			)
+			(justify right bottom)
+		)
+	)
+	(label "pa0"
+		(at 64.77 43.18 180)
+		(effects
+			(font

Commit message: Autosave
Connections:
- net pa2: now also U12.6 (1A2)
- net pa3: now also U12.8 (1A3)
Changed lines of the file:
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@@
+		)
+	)
+	(label "pa3"
+		(at 64.77 50.8 180)
+		(effects
+			(font
+				(size 1.27 1.27)
+				(thickness 0.254)
+				(bold yes)
+			)
+			(justify right bottom)
 		)
 	)
@@
 		)
 	)
+	(label "pa2"
+		(at 64.77 48.26 180)
+		(effects
+			(font
+				(size 1.27 1.27)
+				(thickness 0.254)
+				(bold yes)
+			)
+			(justify right bottom)
+		)
+	)

Commit message: Autosave
Connections:
- net pa0: now also U12.17 (2A0)
- net pa1: now also U12.15 (2A1)
Changed lines of the file:
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@@
+		)
+	)
+	(label "pa0"
+		(at 64.77 53.34 180)
+		(effects
+			(font
+				(size 1.27 1.27)
+				(thickness 0.254)
+				(bold yes)
+			)
+			(justify right bottom)
 		)
 	)
@@
 		(effects
 			(font
+				(size 1.27 1.27)
+				(thickness 0.254)
+				(bold yes)
+			)
+			(justify right bottom)
+		)
+	)
+	(label "pa1"
+		(at 64.77 55.88 180)
+		(effects
+			(font

Commit message: Autosave
Connections:
- net pa2: now also U12.13 (2A2)
- net pa3: now also U12.11 (2A3)
Changed lines of the file:
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@@
+		)
+	)
+	(label "pa3"
+		(at 64.77 60.96 180)
+		(effects
+			(font
+				(size 1.27 1.27)
+				(thickness 0.254)
+				(bold yes)
+			)
+			(justify right bottom)
 		)
 	)
@@
 		(effects
 			(font
+				(size 1.27 1.27)
+				(thickness 0.254)
+				(bold yes)
+			)
+			(justify right bottom)
+		)
+	)
+	(label "pa2"
+		(at 64.77 58.42 180)
+		(effects
+			(font
